File: Head_hub/Head_hub.sch (KiCad schematic (older format))
At the start: 9 parts, among them J1 X_END, J2 LED, J3 RJ45, M1 Fan_3pin, M2 Fan_3pin, M3 Fan_3pin

Commit message: Head_HUB: PCB: Routing done
Parts:
- J1: footprint Connector_JST:JST_XH_S02B-XH-A-1_1x02_P2.50mm_Horizontal -> Connector_JST:JST_XH_B02B-XH-A_1x02_P2.50mm_Vertical
- J2: footprint Connector_JST:JST_XH_S03B-XH-A-1_1x03_P2.50mm_Horizontal -> Connector_JST:JST_XH_B03B-XH-A_1x03_P2.50mm_Vertical
Changed lines of the file:
@@
 F 0 "J1" H 4700 1000 50  0000 L CNN
 F 1 "X_END" H 4700 900 50  0000 L CNN
-F 2 "Connector_JST:JST_XH_S02B-XH-A-1_1x02_P2.50mm_Horizontal" H 4750 1250 50  0001 C CNN
+F 2 "Connector_JST:JST_XH_B02B-XH-A_1x02_P2.50mm_Vertical" H 4750 1250 50  0001 C CNN
 F 3 "~" H 4750 1250 50  0001 C CNN
 	1    4750 1250
@@
 F 0 "J2" H 6350 1150 50  0000 L CNN
 F 1 "LED" H 6350 1050 50  0000 L CNN
-F 2 "Connector_JST:JST_XH_S03B-XH-A-1_1x03_P2.50mm_Horizontal" H 6400 1350 50  0001 C CNN
+F 2 "Connector_JST:JST_XH_B03B-XH-A_1x03_P2.50mm_Vertical" H 6400 1350 50  0001 C CNN
 F 3 "~" H 6400 1350 50  0001 C CNN
 	1    6400 1350
