File: Head_hub/Head_hub.kicad_pcb (KiCad board)
At the start: 2 copper layers, 42.5 x 17 mm, 10 parts, among them J1 X_END, J2 LED, J3 RJ45, M1 Fan_3pin, M2 Fan_3pin, M3 Fan_3pin

Commit message: Head_HUB: PCB: Add QR code with link to GitHub repository
Parts:
- added G***: LOGO, TCY_logo:#QR_3D_PREBO_small, F.Cu at (95.7, 87.5)
