File: Expansion_board/3D_PrEBo.kicad_pcb (KiCad board)
At the start: 2 copper layers, 100 x 84 mm, 78 parts, among them J1 LED, J10 TMC_INPUT, J11 Power_out, J12 Z_Probe, J13 Fan_interconnection_header, J14 X_MIN, J15 Z_MAX, J2 V_IN, J3 RJ45, J4 X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

Commit message: Expansion_board: PCB: Add QR code with link to GitHub repository
Parts:
- added G***: LOGO, TCY_logo:#QR_3D_PREBO, B.Cu at (126.5, 111.5)
